File: pcb/pcb.kicad_sch (KiCad schematic)
At the start: 10 parts, among them U2 DS18B20, U4 nRF52840, U5 LM358

Commit message: pcb sketch updates
Parts:
- removed C1: ~, symbol Library:Ceramic_Cap_-_0.1μ_{gt}7V
- removed Q1: ~, symbol Library:HW5P-1
- removed R1, R2: ~, symbol Library:Resistor_4.7kΩ
- removed R3: ~, symbol Library:Resistor_?1-2kΩ
- removed U1: ~, symbol Library:MMC3419
- removed U4: nRF52840, Package_DFN_QFN:Nordic_AQFN-73-1EP_7x7mm_P0.5mm, symbol MCU_Nordic:nRF52840
- removed U5: LM358, symbol Amplifier_Operational:LM358
- added C1: 0.01μF, GRM155R71C103KA01D:CAPC1005X55N, symbol GRM155R71C103KA01D:GRM155R71C103KA01D
- added C10, C11, C9: 0.1uF, Adafruit nRF52840 Bluefruit Feather Express Rev D:0603-NO, symbol Adafruit nRF52840 Bluefruit Feather Express Rev D-eagle-import:CAP_CERAMIC0603_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
- added C12, C13, C14, C7, C8: 10uF, Adafruit nRF52840 Bluefruit Feather Express Rev D:0805-NO, symbol Adafruit nRF52840 Bluefruit Feather Express Rev D-eagle-import:CAP_CERAMIC0805-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
- added C15, C17, C18, C19, C2, C20, C23, C24, C25, C28, C29, C3, C30, C38: 0.1μF, CL05B104KP5NNNC:CAPC1005X55N, symbol CL05B104KP5NNNC:CL05B104KP5NNNC
- added C16, C21, C22, C26, C27, C31, C37, C4: 10μF, CL21A106KOQNNNG:CAPC2012X140N, symbol CL21A106KOQNNNG:CL21A106KOQNNNG
- added C39: 2.2nF, CGA3E2X7R1H222K080AA:CAPC1608X90N, symbol CGA3E2X7R1H222K080AA:CGA3E2X7R1H222K080AA
- added C5, C6: 22pF, Adafruit nRF52840 Bluefruit Feather Express Rev D:0603-NO, symbol Adafruit nRF52840 Bluefruit Feather Express Rev D-eagle-import:CAP_CERAMIC0603_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
- added D+1, D-1, TP1: TPTP10R, Adafruit nRF52840 Bluefruit Feather Express Rev D:TP10R, symbol Adafruit nRF52840 Bluefruit Feather Express Rev D-eagle-import:TPTP10R
- added D1: RED, Adafruit nRF52840 Bluefruit Feather Express Rev D:CHIPLED_0805_NOOUTLINE, symbol Adafruit nRF52840 Bluefruit Feather Express Rev D-eagle-import:LED0805_NOOUTLINE
- added D2: MBR120, Adafruit nRF52840 Bluefruit Feather Express Rev D:SOD-123, symbol Adafruit nRF52840 Bluefruit Feather Express Rev D-eagle-import:DIODE-SCHOTTKYSO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
- added D3: ORANGE, Adafruit nRF52840 Bluefruit Feather Express Rev D:CHIPLED_0805_NOOUTLINE, symbol Adafruit nRF52840 Bluefruit Feather Express Rev D-eagle-import:LED0805_NOOUTLINE
- added D4: BLUE, Adafruit nRF52840 Bluefruit Feather Express Rev D:CHIPLED_0805_NOOUTLINE, symbol Adafruit nRF52840 Bluefruit Feather Express Rev D-eagle-import:LED0805_NOOUTLINE
- added IC1: GD25Q16, Adafruit nRF52840 Bluefruit Feather Express Rev D:USON8, symbol Adafruit nRF52840 Bluefruit Feather Express Rev D-eagle-import:SPIFLASH_8PINUX
- added L1: DNP, Adafruit nRF52840 Bluefruit Feather Express Rev D:_0805MP, symbol Adafruit nRF52840 Bluefruit Feather Express Rev D-eagle-import:INDUCTOR_0805MP
- added LED1: WS2812B3535, Adafruit nRF52840 Bluefruit Feather Express Rev D:LED3535, symbol Adafruit nRF52840 Bluefruit Feather Express Rev D-eagle-import:WS2812B3535
- added MDBT1: MDBT50, Adafruit nRF52840 Bluefruit Feather Express Rev D:MDBT50, symbol Adafruit nRF52840 Bluefruit Feather Express Rev D-eagle-import:MDBT50
- added Q2, Q4: ~, symbol Library:HW5P-1
- added Q3: DMG2305, Adafruit nRF52840 Bluefruit Feather Express Rev D:SOT23-R, symbol Adafruit nRF52840 Bluefruit Feather Express Rev D-eagle-import:MOSFET-P
- added R1, R2: 22, Adafruit nRF52840 Bluefruit Feather Express Rev D:0603-NO, symbol Adafruit nRF52840 Bluefruit Feather Express Rev D-eagle-import:RESISTOR_0603_NO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
- added R10, R6, R9: 1K, Adafruit nRF52840 Bluefruit Feather Express Rev D:0603-NO, symbol Adafruit nRF52840 Bluefruit Feather Express Rev D-eagle-import:RESISTOR_0603_NO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
- added R11, R14, R17, R20: 39K, RC0402FR-0739KL:RESC1005X40N, symbol RC0402FR-0739KL:RC0402FR-0739KL
- added R12, R15, R18, R21: 45K, RC0402FR-0745K3L:RESC1005X40N, symbol RC0402FR-0745K3L:RC0402FR-0745K3L
- added R13, R16, R19, R3: 20, CRCW251220R0FKEG:RESC6331X70N, symbol CRCW251220R0FKEG:CRCW251220R0FKEG
- added R22, R4, R5: 4.7K, RC0402JR-074K7L:RESC1005X40N, symbol RC0402JR-074K7L:RC0402JR-074K7L
- added R23: 30K, ERA2AEB303X:RES_ERA2AEB303X, symbol ERA2AEB303X:ERA2AEB303X
- added R24: 100K, RC0402FR-07100KL:RESC1005X40, symbol RC0402FR-07100KL:RC0402FR-07100KL
- added R7: 100K, Adafruit nRF52840 Bluefruit Feather Express Rev D:RESPACK_4X0603, symbol Adafruit nRF52840 Bluefruit Feather Express Rev D-eagle-import:RESISTOR_4PACK
- added R8: 4.7K, Adafruit nRF52840 Bluefruit Feather Express Rev D:0603-NO, symbol Adafruit nRF52840 Bluefruit Feather Express Rev D-eagle-import:RESISTOR_0603_NO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
- added SW1, SW2: KMR2, Adafruit nRF52840 Bluefruit Feather Express Rev D:BTN_KMR2_4.6X2.8, symbol Adafruit nRF52840 Bluefruit Feather Express Rev D-eagle-import:SWITCH_TACT_SMT4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
- added SWC1, SWD1: TPTP12R, Adafruit nRF52840 Bluefruit Feather Express Rev D:TP12R, symbol Adafruit nRF52840 Bluefruit Feather Express Rev D-eagle-import:TPTP12R
- added U1: MPU-6050, Sensor_Motion:InvenSense_QFN-24_4x4mm_P0.5mm, symbol Sensor_Motion:MPU-6050
- added U10, U12, U14, U4: INA333xxDGK, Package_SO:VSSOP-8_3.0x3.0mm_P0.65mm, symbol Amplifier_Instrumentation:INA333xxDGK
- added U11, U13, U5, U9: MCP6002-I/SN, SOIC8-N_MC_MCH, symbol 2024-11-12_18-15-18:MCP6002-I_SN
- added U20: MCP6001-OT, Package_TO_SOT_SMD:SOT-23-5, symbol Amplifier_Operational:MCP6001-OT
- added U6: CS5523-ASZ, CIR-SSOP-24, symbol 2024-11-11_22-44-29:CS5523-ASZ
- added U7: AP2112(3.3V), Adafruit nRF52840 Bluefruit Feather Express Rev D:SOT23-5, symbol Adafruit nRF52840 Bluefruit Feather Express Rev D-eagle-import:VREG_SOT23-5
- added U8: MCP73831T-2ACI/OT, Adafruit nRF52840 Bluefruit Feather Express Rev D:SOT23-5, symbol Adafruit nRF52840 Bluefruit Feather Express Rev D-eagle-import:MCP73831/2
- added X1: 2x5 0.05", Adafruit nRF52840 Bluefruit Feather Express Rev D:2X05_1.27MM_BOX_POSTS, symbol Adafruit nRF52840 Bluefruit Feather Express Rev D-eagle-import:JTAG-CORTEXBOXPO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
- added X2: 4u20329, Adafruit nRF52840 Bluefruit Feather Express Rev D:4UCONN_20329_V2, symbol Adafruit nRF52840 Bluefruit Feather Express Rev D-eagle-import:USB_MICRO_20329_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
- added X3: JSTPH, Adafruit nRF52840 Bluefruit Feather Express Rev D:JSTPH2, symbol Adafruit nRF52840 Bluefruit Feather Express Rev D-eagle-import:CON_JST_PH_2PIN
- added Y1: 32.768, Adafruit nRF52840 Bluefruit Feather Express Rev D:XTAL3215, symbol Adafruit nRF52840 Bluefruit Feather Express Rev D-eagle-import:XTAL-3.2X1.5
Connections:
- net GND: now also C1.2, C10.1, C11.1, C12.1, C13.1, C14.1, C15.2, C16.2, C17.2, C18.1, C19.1, C2.1, C20.1, C21.2, C22.2, C23.2, C24.1, C25.1, C26.2, C27.2, C28.2, C29.1, C3.1, C30.1, C31.2, C37.2, C38.1, C39.2, C4.2, C5.2, C6.2, C7.1, C8.1, C9.1, D1.C, IC1.4 (VSS), LED1.4 (GND), MDBT1.1 (GND@1), MDBT1.15 (GND@15), MDBT1.2 (GND@2), MDBT1.33 (GND@33), MDBT1.55 (GND@55), R10.2, R22.2, R23.2, R4.2, R5.2, R7.3 (1), R7.8 (2), R8.2, SW1.A (P), SW1.A' (P1), SW2.A (P), SW2.A' (P1), U1.1 (CLKIN), U1.11 (FSYNC), U1.18 (GND), U10.4 (V-), U11.4 (VSS), U12.4 (V-), U13.4 (VSS), U14.4 (V-), U4.4 (V-), U5.4 (VSS), U6.1 (AGND), U6.15 (DGND), U6.19 (AIN4-), U6.21 (AIN2-), U6.23 (VREF-), U6.4 (AIN1-), U6.6 (AIN3-), U7.2 (GND), U8.2 (VSS), U9.4 (VSS), X1.3 (GND@1), X1.5 (GND@2), X1.7 (KEY), X1.9 (GNDDETECT), X2.BASE@1 (GND), X2.BASE@2 (GND), X2.GND, X2.SPRT@1 (GND), X2.SPRT@2 (GND), X2.SPRT@3 (GND), X2.SPRT@4 (GND), X3.1
- net A3: now reaches U3. (OUT)
- net A3: now also MDBT1.13 (P0.28/AIN4), R22.1
- net A2: now reaches U2.2 (DQ)
- net A2: now also MDBT1.14 (P0.30/AIN6)
- net VCC renamed 3.3V
- net 3.3V: now also C1.1, C10.2, C14.2, C15.1, C17.1, C19.2, C22.1, C23.1, C24.2, C27.1, C28.1, C29.2, C3.2, C37.1, C38.2, C4.1, C7.2, C9.2, IC1.8 (VCC), L1.1, LED1.2 (VDD), MDBT1.28 (VDD), MDBT1.30 (VDDH), Q2.1 (Vdd), Q4.1 (Vdd), R24.1, U1.13 (VDD), U1.8 (VLOGIC), U10.7 (V+), U11.8 (VDD), U12.7 (V+), U13.8 (VDD), U14.7 (V+), U4.7 (V+), U5.8 (VDD), U6.16 (VD+), U6.2 (VA+), U7.5 (OUT), U9.8 (VDD), X1.1 (VCC)
- new net: R12.1, U9.1 (VOUTA)
- new net: C16.1, R11.2, U9.3 (VINA+)
- new net: C18.2, R12.2, U9.6 (VINB-)
- new net: C30.2, R21.2, U13.6 (VINB-)
- new net: R17.1, U12.6
- new net: C26.1, R17.2, U11.3 (VINA+)
- new net: R15.1, U5.1 (VOUTA)
- new net: C21.1, R14.2, U5.3 (VINA+)
- new net: C20.2, R15.2, U5.6 (VINB-)
- new net: R18.1, U11.1 (VOUTA)
- new net: C25.2, R18.2, U11.6 (VINB-)
- new net: MDBT1.52 (P0.09/NFC1), TP1.TP
- new net: D3.C, R9.1
- new net: R23.1, R24.2, U20.3 (+)
- new net: C12.2, D2.C, Q3.2 (S), R7.7 (2), U7.1 (IN)
- new net: D+1.TP, R1.1, X2.D+
- new net: D4.C, R10.1
- new net: C2.2, U1.10 (REGOUT)
- new net: C39.1, U1.20 (CPOUT)
- new net: R3.1, U4.1 (Rg)
- new net: R3.2, U4.8 (Rg)
- new net: R16.1, U12.1 (Rg)
- new net: R16.2, U12.8 (Rg)
- new net: R13.1, U10.1 (Rg)
- new net: R14.1, U10.6
- new net: R13.2, U10.8 (Rg)
- new net: D1.A, R6.2
- new net: R9.2, U8.1 (STAT)
- new net: R8.1, U8.5 (PROG)
- new net: D-1.TP, R2.1, X2.D-
- new net: R21.1, U13.1 (VOUTA)
- new net: C31.1, R20.2, U13.3 (VINA+)
- new net: U20.1, U20.4 (-), U6.24 (VREF+)
- new net: C5.1, MDBT1.17 (P0.00/XL1), Y1.P$1
- new net: C6.1, MDBT1.18 (P0.01/XL2), Y1.P$2
- new net: R19.1, U14.1 (Rg)
- new net: R19.2, U14.8 (Rg)
- new net: R11.1, U4.6
- new net: R20.1, U14.6
- new net A0: MDBT1.20 (P0.04/AIN2), Q4.2 (Vout), R4.1
- new net A1: MDBT1.21 (P0.05/AIN3), Q2.2 (Vout), R5.1
- new net A4: MDBT1.11 (P0.02/AIN0)
- new net A5: MDBT1.9 (P0.03/AIN1)
- new net AREF: C11.2, MDBT1.12 (P0.31/AIN7)
- new net D10: MDBT1.16 (P0.27)
- new net D11: MDBT1.22 (P0.06)
- new net D12: MDBT1.24 (P0.08)
- new net D13: MDBT1.26 (P1.09)
- new net D2: MDBT1.54 (P0.10/NFC2)
- new net D5: MDBT1.25 (P1.08)
- new net D6: MDBT1.23 (P0.07)
- new net D9: MDBT1.19 (P0.26)
- new net DCCH: L1.2, MDBT1.31 (DCCH)
- new net EEG1 OUT: U6.3 (AIN1+), U9.7 (VOUTB)
- new net EEG1+: U4.3 (+)
- new net EEG1-: U4.2 (-)
- new net EEG2 OUT: U5.7 (VOUTB), U6.22 (AIN2+)
- new net EEG2+: U10.3 (+)
- new net EEG2-: U10.2 (-)
- new net EEG3 OUT: U13.7 (VOUTB), U6.5 (AIN3+)
- new net EEG3+: U14.3 (+)
- new net EEG3-: U14.2 (-)
- new net EEG4 OUT: U11.7 (VOUTB), U6.20 (AIN4+)
- new net EEG4+: U12.3 (+)
- new net EEG4-: U12.2 (-)
- new net EN: R7.2 (1), U7.3 (EN)
- new net LED1: MDBT1.8 (P1.15), R6.1
- new net LED2: D4.A, MDBT1.3 (P1.10)
- new net MISO: MDBT1.39 (P0.15), U6.14 (SDO)
- new net MOSI: MDBT1.37 (P0.13), U6.10 (SDI)
- new net NEOPIX: LED1.1 (DI), MDBT1.38 (P0.16)
- new net QSPI_CS: IC1.1 (SSEL), MDBT1.44 (P0.20)
- new net QSPI_DATA0: IC1.5 (MOSI), MDBT1.41 (P0.17)
- new net QSPI_DATA1: IC1.2 (MISO), MDBT1.46 (P0.22)
- new net QSPI_DATA2: IC1.3 (WP#/IO2), MDBT1.45 (P0.23)
- new net QSPI_DATA3: IC1.7 (HOLD#/IO3), MDBT1.43 (P0.21)
- new net QSPI_SCK: IC1.6 (SCK), MDBT1.42 (P0.19)
- new net RESET: MDBT1.40 (P0.18/RESET), SW1.B (S), SW1.B' (S1), X1.10 (NRESET)
- new net RXD: MDBT1.48 (P0.24)
- new net SCK: MDBT1.36 (P0.14)
- new net SCL: MDBT1.27 (P0.11), U1.23 (SCL)
- new net SDA: MDBT1.29 (P0.12), U1.24 (SDA)
- new net SWCLK: MDBT1.53 (SWDCLK), SWC1.TP, X1.4 (SWDCLK)
- new net SWDIO: MDBT1.51 (SWDIO), SWD1.TP, X1.2 (SWDIO)
- new net SWITCH: MDBT1.50 (P1.02), SW2.B (S), SW2.B' (S1)
- new net SWO: MDBT1.47 (P1.00), X1.6 (SWO)
- new net TXD: MDBT1.49 (P0.25)
- new net USBD+: MDBT1.35 (D+), R1.2
- new net USBD-: MDBT1.34 (D-), R2.2
- new net VBAT: C13.2, Q3.3 (D), R7.4 (1), U8.3 (VBAT), X3.2
- new net VBUS: C8.2, D2.A, D3.A, MDBT1.32 (VBUS), Q3.1 (G), R7.1, U8.4 (VDD), X2.VBUS
- new net VDIV: MDBT1.10 (P0.29/AIN5), R7.5 (2), R7.6 (2)
Other:
- note added: "1.0K = 1000mA"
- note added: "10K = 100mA"
- note added: "16MBIT QSPI FLASH"
- note added: "2.0K = 500mA"
- note added: "5.0K = 200mA"
- note added: "Accel / Gyro"
- note added: "DECOUPLING CAPS"
- note added: "Dropout Voltage (25°C): 100mA: ~250/~40mV 300mA: ~300/~125mV 600mA: ~375/~260mV"
- note added: "Dynamic VIN selection: VBUS (USB) will override VBAT (LIPO) via D5 when both are present."
- note added: "EEG circuit 1"
- note added: "EEG circuit 2"
- note added: "EEG circuit 3"
- note added: "Heart rate sensor"
- note added: "INDICATOR LEDS"
- note added: "JST PH LIPO INPUT"
- note added: "LIPO CHARGING"
- note added: "MICRO USB"
- note added: "NEOPIXEL"
- note added: "POWER AND FILTERING (600mA Output)"
- note added: "Phototransistor 1"
- note added: "Phototransistor 2"
- note added: "Place 10uH for DC/DC"
- note added: "RESET/USER SWITCHES"
- note added: "SWD DEBUGGER"
- note added: "Thermometer"
- note added: "To charge the LIPO, insert the battery in the JST PH connector and connect USB at the same time."
- moved on the sheet: U2, U3
