File: pcb/pcb.kicad_sch (KiCad schematic)
At the start: 114 parts, among them IC1 GD25Q16, J1 10118194-0001LF, Q3 DMG2305, SW1 KMR2, SW2 KMR2, U1 MPU-6050, U10 INA333xxDGK, U11 LM358DT, U12 INA333xxDGK, U13 LM358DT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

Commit message: pcb updates
Parts:
- removed D+1, D-1, TP1: TPTP10R, Adafruit nRF52840 Bluefruit Feather Express Rev D:TP10R, symbol Adafruit nRF52840 Bluefruit Feather Express Rev D-eagle-import:TPTP10R
- removed L1: DNP, Adafruit nRF52840 Bluefruit Feather Express Rev D:_0805MP, symbol Adafruit nRF52840 Bluefruit Feather Express Rev D-eagle-import:INDUCTOR_0805MP
- removed LED1: WS2812B3535, Adafruit nRF52840 Bluefruit Feather Express Rev D:LED3535, symbol Adafruit nRF52840 Bluefruit Feather Express Rev D-eagle-import:WS2812B3535
- removed Q2, Q4: ~, symbol Library:HW5P-1
- removed R7: 100K, Library:RESC2012X60N, symbol Adafruit nRF52840 Bluefruit Feather Express Rev D-eagle-import:RESISTOR_4PACK
- removed SW1, SW2: KMR2, Adafruit nRF52840 Bluefruit Feather Express Rev D:BTN_KMR2_4.6X2.8, symbol Adafruit nRF52840 Bluefruit Feather Express Rev D-eagle-import:SWITCH_TACT_SMT4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
- removed SWC1, SWD1: TPTP12R, Adafruit nRF52840 Bluefruit Feather Express Rev D:TP12R, symbol Adafruit nRF52840 Bluefruit Feather Express Rev D-eagle-import:TPTP12R
- removed U3: ~, symbol Library:SEN-11574
- removed X3: JSTPH, Adafruit nRF52840 Bluefruit Feather Express Rev D:JSTPH2, symbol Adafruit nRF52840 Bluefruit Feather Express Rev D-eagle-import:CON_JST_PH_2PIN
- added D5: 2659, Library:2659, symbol Library:2659
- added J2: 0533980271, Library:MOLEX_0533980271, symbol Library:0533980271
- added R36, R37, R38, R7: 100K, Library:RESC2012X60N, symbol Library:Resistor
- added SW1, SW2: KMR223G LFG, Library:KMR2_G_CNK, symbol Library:KMR223G_LFG
- added U3: ~, Library:Sensors, symbol Library:sensors
- C1: footprint GRM155R71C103KA01D:CAPC1005X55N -> Library:CAPC2012X95N
- C15, C18, C24, C25: value 100nF -> 0.1μF; footprint CL05B104KP5NNNC:CAPC1005X55N -> Library:CAPC2012X88N
- C16, C31, C4: value 100nF -> 0.1μF; footprint CL21A106KOQNNNG:CAPC2012X140N -> Library:CAPC2012X88N
- C22: value 2nF -> 2.2nF; footprint CL21A106KOQNNNG:CAPC2012X140N -> Library:CAP_CL21_SAM
- C23, C30: footprint CL05B104KP5NNNC:CAPC1005X55N -> Library:CAP_0805J_AVX
- C29: value 2nF -> 2.2nF; footprint CL05B104KP5NNNC:CAPC1005X55N -> Library:CAP_CL21_SAM
- C32, C41: value 2nF -> 2.2nF; footprint (none) -> Library:CAP_CL21_SAM
- C33, C42: footprint (none) -> Library:CAP_0805J_AVX
- C34: value 100nF -> 0.1μF; footprint (none) -> Library:CAPC2012X88N
- C5, C6: footprint Adafruit nRF52840 Bluefruit Feather Express Rev D:0603-NO -> Library:CAPC220145_88N_KEM
- D1, D3, D4: footprint Adafruit nRF52840 Bluefruit Feather Express Rev D:CHIPLED_0805_NOOUTLINE -> Library:WL-SMCW_0805
- D2: footprint Adafruit nRF52840 Bluefruit Feather Express Rev D:SOD-123 -> Library:SDO_SOD-123FL498_OSI
- IC1: footprint Adafruit nRF52840 Bluefruit Feather Express Rev D:USON8 -> Library:SOIC127P600X175-8N
- MDBT1: footprint Adafruit nRF52840 Bluefruit Feather Express Rev D:MDBT50 -> Library:MDBT50Q-U
- Q3: footprint Adafruit nRF52840 Bluefruit Feather Express Rev D:SOT23-R -> Library:SOT91P240X110-3N_DMG2305UX-7
- R1, R2: footprint Adafruit nRF52840 Bluefruit Feather Express Rev D:0603-NO -> Library:RESC2012X60N
- R11, R20: value 4.5K -> 4.7K; footprint RC0402FR-0739KL:RESC1005X40N -> Library:RESC2012X60N
- R12, R18: value 2.25K -> 2.2K; footprint RC0402FR-0745K3L:RESC1005X40N -> Library:RESC2012X60N
- R13: value 2.25K -> 2.2K
- R14, R19, R3, R32: value 20 -> 22; footprint Library:20Ohm-RESC2012X60N -> Library:RESC2012X60N
- R15: value 4.5K -> 4.7K; footprint RC0402FR-0745K3L:RESC1005X40N -> Library:RESC2012X60N
- R16: value 3.75K -> 3.74K
- R17: value 3.75K -> 3.74K; footprint RC0402FR-0739KL:RESC1005X40N -> Library:RESC2012X60N
- R21: value 3.75K -> 3.74K; footprint RC0402FR-0745K3L:RESC1005X40N -> Library:RESC2012X60N
- R28, R29, R30, R34, R35: value 3.75K -> 3.74K; footprint (none) -> Library:RESC2012X60N
- R31: value 2.25K -> 2.2K; footprint (none) -> Library:RESC2012X60N
- R33: value 4.5K -> 4.7K; footprint (none) -> Library:RESC2012X60N
- U7: footprint Adafruit nRF52840 Bluefruit Feather Express Rev D:SOT23-5 -> Library:SOT_RG1_DIO
- U8: footprint Adafruit nRF52840 Bluefruit Feather Express Rev D:SOT23-5 -> Library:SOT-23-5_MC_MCH
- X1: footprint Adafruit nRF52840 Bluefruit Feather Express Rev D:2X05_1.27MM_BOX_POSTS -> Library:2X05_1.27MM_BOX_POSTS
- Y1: footprint Adafruit nRF52840 Bluefruit Feather Express Rev D:XTAL3215 -> Library:XTAL_SC32S-7PF20PPM_EPS
Connections:
- net 3.3V: now also D5.4 (VDD), U3.1 (Photo1_VDD), U3.3 (Photo2_VDD), U3.5 (HRT_+V)
- net A0: now also U3.2 (Photo1_Vout)
- net A1: now also U3.4 (Photo1_Vout)
- net A3: now also U3.6 (HRT_OUT)
- net EEG1+: now also U3.8 (EEG1+)
- net EEG2+: now also U3.9 (EEG2+)
- net EEG3+: now also U3.10 (EEG3+)
- net EEG4+: now also U3.11 (EEG4+)
- net EN: now also R36.2
- net GND: now also D5.2 (VSS), J2.2, R38.2, R7.2, SW1.3, SW2.3, U3.12 (EEG_GND), U3.7 (HRT_GND)
- net NEOPIX: now also D5.3 (DIN)
- net RESET: now also SW1.2
- net SWITCH: now also SW2.2
- net VBAT: now also J2.1, R37.1
- net VBUS: now also R7.1
- net VDIV: now also R37.2, R38.1
- net at C12.2, D2.C, Q3.2 (S)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: now also R36.1
- net at C5.1, MDBT1.17 (P0.00/XL1): now also Y1.1 (P$1); no longer Y1.P$1
- net at C6.1, MDBT1.18 (P0.01/XL2): now also Y1.2 (P$2); no longer Y1.P$2
- no-connect marks 39 -> 41
Other:
- moved on the sheet: R22

Commit message: pcb updates
Parts:
- removed R23: 30K, Library:RESC2012X65N, symbol ERA2AEB303X:ERA2AEB303X
- removed R24: 100K, Library:RESC2012X60N, symbol RC0402FR-07100KL:RC0402FR-07100KL
- removed U20: MCP6001-OT, Package_TO_SOT_SMD:SOT-23-5, symbol Amplifier_Operational:MCP6001-OT
- added U14: ISL21080DIH309Z-TK, Library:P3_064_INR, symbol Library:ISL21080DIH309Z-TK
Connections:
- net 3.3V: now also U14.1 (VIN)
- net GND: now also J1.SH1 (SHIELD), J1.SH2 (SHIELD__1), J1.SH3 (SHIELD__2), J1.SH4 (SHIELD__3), J1.SH5 (SHIELD__4), J1.SH6 (SHIELD__5), J2.S1 (SHIELD), J2.S2 (SHIELD__1), U14.3 (GND)
- net at U6.24 (VREF+): now also U14.2 (VOUT)
- net USBD+ renamed USB_P
- net USBD- renamed USB_N
- no-connect marks 41 -> 47

Commit message: pcb updates
Parts:
- added C43, C44: 0.1μF, Library:CAPC2012X88N, symbol CL05B104KP5NNNC:CL05B104KP5NNNC
- added C45: 10μF, Library:CAPC2012X88N, symbol CL21A106KOQNNNG:CL21A106KOQNNNG
- added U16, U17, U18, U19: ~, Library:EEG_DEBUG, symbol Library:EEG_debug
Connections:
- net 3.3V: now also C44.2, C45.1
- net EEG1 OUT: now also U19.1 (EEG_DEBUG)
- net EEG2 OUT: now also U18.1 (EEG_DEBUG)
- net EEG3 OUT: now also U17.1 (EEG_DEBUG)
- net EEG4 OUT: now also U16.1 (EEG_DEBUG)
- net GND: now also C43.1, C44.1, C45.2
- net at U14.2 (VOUT), U6.24 (VREF+): now also C43.2
