File: pcb/pcb.kicad_pcb (KiCad board)
At the start: 2 copper layers, 109 parts, among them IC1 GD25Q16, J1 10118194-0001LF, J2 0533980271, Q3 DMG2305, SW1 KMR223G LFG, SW2 KMR223G LFG, U1 MPU-6050, U10 INA333xxDGK, U11 LM358DT, U12 INA333xxDGK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

Commit message: pcb updates
Parts:
- moved R23 107.8 mm to (148.2, 90.1)
- moved R24 107.8 mm to (144.7, 90.1)
- moved U20 107.8 mm to (151.7, 89.5)
- moved C29 107.2 mm to (131.4, 90.8), turned to 90 degrees
- moved U6 106.4 mm to (148.8, 97.0)
- moved C27 105.2 mm to (135.0, 87.2), turned to 0 degrees
- moved R30 104.9 mm to (131.4, 94.2), turned to 90 degrees
- moved R18 102.9 mm to (131.4, 98.7), turned to -90 degrees
- moved U11 101.3 mm to (135.3, 92.3), turned to 90 degrees
- moved C25 99.6 mm to (134.0, 98.7), turned to -90 degrees
- moved R19 99.3 mm to (132.7, 102.5), turned to 90 degrees
- moved C35 98.6 mm to (136.4, 124.4)
- moved C36 98.6 mm to (132.6, 124.4), turned to 180 degrees
- moved R33 98.6 mm to (139.7, 125.1)
- moved U12 98.6 mm to (134.0, 121.3)
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Routing:
- net GND: track 0.00 -> 319.9 mm
- net 3.3V: track 0.00 -> 278.4 mm, vias 0 -> 21
- net /MISO: track 0.00 -> 119.3 mm, vias 0 -> 6
- net /SCK: track 0.00 -> 99.6 mm, vias 0 -> 4
- net /USBD+: track 0.00 -> 94.1 mm, vias 0 -> 4
- net /MOSI: track 0.00 -> 92.1 mm, vias 0 -> 2
- net /USBD-: track 0.00 -> 87.5 mm, vias 0 -> 4
- net /A3: track 0.00 -> 85.6 mm, vias 0 -> 4
- net /EEG1 OUT: track 0.00 -> 83.4 mm, vias 0 -> 6
- net /A0: track 0.00 -> 82.2 mm, vias 0 -> 6
- net /RESET: track 0.00 -> 81.0 mm, vias 0 -> 4
- net /ADC CS: track 0.00 -> 75.7 mm, vias 0 -> 2
- net /SDA: track 0.00 -> 72.6 mm, vias 0 -> 8
- net VBUS: track 0.00 -> 71.0 mm, vias 0 -> 2
- net /SCL: track 0.00 -> 65.1 mm, vias 0 -> 8
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- added copper zone on B.Cu, net 3.3V
- added copper zone on F.Cu, net GND
Other:
- board outline added: 73.7 x 44.5 mm
- board text added: "EEG-"
- board text added: "EEG1"
- board text added: "EEG2"
- board text added: "EEG3"
- board text added: "EEG4"
- board text added: "HRT"
- board text added: "HRT+"
- board text added: "HRT-"
- board text added: "P1+"
- board text added: "P1-"
- board text added: "P2+"
- board text added: "P2-"

Commit message: pcb updates
Parts:
- removed R23: 30K, Library:RESC2012X65N
- removed R24: 100K, Library:RESC2012X60N
- removed U20: MCP6001-OT, Package_TO_SOT_SMD:SOT-23-5
- added U14: ISL21080DIH309Z-TK, Library:P3_064_INR, F.Cu at (147.0, 88.5)
- moved R2 2.24 mm to (167.0, 94.0)
- moved R1 2.24 mm to (163.2, 94.1), turned to 0 degrees
- moved R22 0.63 mm to (139.7, 113.7)
Connections:
- net /USBD+ renamed /USB_P
- net /USBD- renamed /USB_N
- J1 pad SH1: unconnected-(J1-SHIELD-PadSH1) -> GND
- J1 pad SH2: unconnected-(J1-SHIELD__1-PadSH2) -> GND
- J1 pad SH3: unconnected-(J1-SHIELD__2-PadSH3) -> GND
- J1 pad SH4: unconnected-(J1-SHIELD__3-PadSH4) -> GND
- J1 pad SH5: unconnected-(J1-SHIELD__4-PadSH5) -> GND
- J1 pad SH6: unconnected-(J1-SHIELD__5-PadSH6) -> GND
- J2 pad S1: unconnected-(J2-SHIELD-PadS1) -> GND
- J2 pad S2: unconnected-(J2-SHIELD__1-PadS2) -> GND
Routing:
- net GND: track 319.9 -> 39.4 mm, vias 0 -> 51
- net 3.3V: track 278.4 -> 253.5 mm, vias 21 -> 19
- net VBUS: track 71.0 -> 55.9 mm
- net /A0: track 82.2 -> 68.9 mm
- net /SCL: track 65.1 -> 75.8 mm
- net /MOSI: track 92.1 -> 100.4 mm
- net VBAT: track 45.7 -> 38.0 mm
- net /ADC CS: track 75.7 -> 83.2 mm
- net /SCK: track 99.6 -> 106.8 mm
- net /USB_P: track 94.1 -> 88.2 mm, vias 4 -> 2
- net Net-(U20-+): track 5.81 -> 0.00 mm
- net /A3: track 85.6 -> 91.1 mm, vias 4 -> 6
- net /SWITCH: track 22.5 -> 26.3 mm
- net /SWCLK: track 40.9 -> 37.4 mm
- net /MISO: track 119.3 -> 122.1 mm
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- added copper zone on B.Cu, net GND

Commit message: pcb updates
Parts:
- added C43: 0.1μF, Library:CAPC2012X88N, F.Cu at (150.7, 88.8)
- added C44: 0.1μF, Library:CAPC2012X88N, F.Cu at (145.8, 91.3)
- added C45: 10μF, Library:CAPC2012X88N, F.Cu at (144.0, 87.8)
- added U16: ~, Library:EEG_DEBUG, F.Cu at (150.1, 122.2)
- added U17: ~, Library:EEG_DEBUG, F.Cu at (129.2, 91.8)
- added U18: ~, Library:EEG_DEBUG, F.Cu at (173.2, 123.8)
- added U19: ~, Library:EEG_DEBUG, F.Cu at (196.0, 123.7)
- moved SW2 0.88 mm to (193.5, 88.9)
- moved SW1 0.40 mm to (189.5, 88.9)
- moved U14 0.29 mm to (147.0, 88.2)
Routing:
- net VBAT: track 38.0 -> 50.6 mm, vias 2 -> 6
- net /MISO: track 122.1 -> 112.5 mm
- net 3.3V: track 253.5 -> 262.4 mm, vias 19 -> 21
- net /SCL: track 75.8 -> 68.7 mm
- net /A3: track 91.1 -> 84.7 mm
- net /MOSI: track 100.4 -> 96.0 mm
- net /SWO: track 49.1 -> 53.5 mm
- net /EEG2+: track 26.3 -> 22.2 mm
- net /SDA: track 75.4 -> 71.7 mm
- net /EEG3 OUT: track 19.5 -> 23.1 mm
- net GND: track 39.4 -> 36.0 mm, vias 51 -> 56
- net /SCK: track 106.8 -> 103.6 mm
- net /SWCLK: track 37.4 -> 34.2 mm
- net /EEG2 OUT: track 52.4 -> 55.4 mm
- net /SWITCH: track 26.3 -> 23.4 mm
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